File: PCBs/MITCH_2021-48/PSPS_AVNC_SRD_CS_combined-2021-02-07.brd (EAGLE design)
At the start: 129.8 x 132.6 mm, 48 parts, among them J1 A-1JB, U0-C STM32F411CEUX, U0-S TPS62202, U1-S ICM-20948

Commit message: Finished Flight Ready PCB Draft
Parts:
- added JP2: (no value), pinhead:1X05
- added LD1, LD2: (no value), adafruit:CHIP-LED0805
- added R11, R12, R17: 10k, resistor:M0805
- added R13, R14, R15, R16: TBD, resistor:M0805
- added S2: (no value), switch-omron:B3F-10XX
- added U$18, U$19: TLC5916SOIC-16, Computer2:SOIC127P600X175-16N
- added U$20, U$21: TLC5926TSSOP, Computer2:SOP65P640X120-24N
- moved LED1 195.0 mm to (76.8, 30.2)
- moved LED2 195.0 mm to (70.5, 30.2)
- moved LED3 195.0 mm to (64.2, 30.2)
- moved LED4 195.0 mm to (58.0, 30.2)
- moved R10 195.0 mm to (38.5, 11.2)
- moved R8 195.0 mm to (45.8, 23.8)
- moved R9 195.0 mm to (38.5, 17.5)
- moved U$17 195.0 mm to (38.8, 24.5)
- moved JP1 188.0 mm to (65.0, 37.0)
- moved C1 10.0 mm to (4.50, -7.75)
- moved C10 10.0 mm to (-9.25, -25.5)
- moved C2 10.0 mm to (-51.8, 0.00)
- moved C3 10.0 mm to (-27.2, -18.0)
- moved C4 10.0 mm to (-20.8, -18.0)
- moved C5 10.0 mm to (-17.6, -21.0)
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Connections:
- new net N$10: R15.1, U$20.23
- new net N$11: R16.1, U$21.23
- new net N$12: U$19.5
- new net N$13: U$19.6
- new net N$14: U$19.7
- new net N$15: U$19.8
- new net N$16: U$19.12
- new net N$17: U$19.11
- new net N$18: U$19.10
- new net N$19: U$19.9
- new net N$20: U$18.5
- new net N$21: U$18.6
- new net N$22: U$18.7
- new net N$23: U$18.8
- new net N$24: U$18.12
- new net N$25: U$18.11
- new net N$26: U$18.10
- new net N$27: U$18.9
- new net N$28: U$20.20
- new net N$29: U$20.19
- new net N$30: U$20.18
- new net N$31: U$20.17
- new net N$32: U$20.16
- new net N$33: U$20.15
- new net N$34: U$20.14
- new net N$35: U$20.13
- new net N$36: U$21.20
- new net N$37: U$21.19
- new net N$38: U$21.18
- new net N$39: U$21.17
- new net N$40: U$21.16
- new net N$41: U$21.15
- new net N$42: U$21.14
- new net N$43: U$21.13
- new net N$44: U$21.5
- new net N$45: U$21.6
- new net N$46: U$21.7
- new net N$47: U$21.8
- new net N$48: U$21.9
- new net N$49: U$21.10
- new net N$50: U$21.11
- new net N$51: U$21.12
- new net N$52: U$20.5
- new net N$53: U$20.6
- new net N$54: U$20.7
- new net N$55: U$20.8
- new net N$56: U$20.9
- new net N$57: U$20.10
- new net N$58: U$20.11
- new net N$59: U$20.12
- new net N$6: LD1.C, R11.1
- new net N$60: R17.1, S2.4
- new net N$7: LD2.C, R12.1
- new net N$8: R13.1, U$18.15
- new net N$9: R14.1, U$19.15
- net 3V3: now also JP2.1, S2.1, U$18.16, U$19.16, U$20.24, U$21.24
- net BUTTON_IN: now also S2.3, U0-C.32; no longer U0-C.33
- net BUZZER_OUT: now also U0-C.33; no longer U0-C.32
- net GND: now also JP2.5, R11.2, R12.2, R13.2, R14.2, R15.2, R16.2, R17.2, U$18.1, U$18.13, U$19.1, U$19.13, U$20.1, U$20.21, U$21.1, U$21.21
- net LD1: now also LD1.A
- net LD2: now also LD2.A
- net SPI2B_LE: now also U$18.4, U$19.4, U$20.4, U$21.4
- net SPI2B_MOSI: now also U$18.2, U$19.2, U$20.2, U$21.2
- net SPI2_CS0: now also U$4.4; no longer U$4.13
- net SPI2_CS2: now also U$4.13; no longer U$4.4
- net SPI2_SCK0: now also U$18.3, U$19.3, U$20.3, U$4.6; no longer U$4.11
- net SPI2_SCK2: now also U$4.11; no longer U$4.6
- net SPI2_SCK3: now also U$21.3
- net SWCLK: now also JP2.3
- net SWDIO: now also JP2.4
- net SWO: now also JP2.2
Routing:
- net 3V3: track 93.8 -> 121.6 mm
- net GND: track 215.7 -> 239.6 mm, vias 18 -> 21
- net EXT-ANT: track 21.2 -> 0.00 mm, vias 1 -> 0
- net SPI2_SCK0: track 0.82 -> 18.7 mm
- net SPI2B_LE: track 1.07 -> 17.0 mm, vias 1 -> 3
- net N$10: track 0.00 -> 12.6 mm
- net SWO: track 0.00 -> 12.2 mm
- net SPI2B_MOSI: track 1.07 -> 12.1 mm, vias 1 -> 3
- net SWCLK: track 0.00 -> 10.7 mm
- net SPI2_SCK3: track 0.80 -> 11.3 mm
- net SWDIO: track 3.64 -> 11.9 mm
- net SPI2_SCK: track 35.9 -> 44.1 mm
- net BUTTON_IN: track 4.00 -> 11.6 mm
- net N$44: track 0.00 -> 7.50 mm
- net N$36: track 0.00 -> 7.50 mm
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- added copper zone on layer 2, net GND
Other:
- board size 129.8 x 132.6 mm -> 132.6 x 129.8 mm
