File: PCBs/MITCH_2021-48/PSPS_AVNC_SRD_CS_combined-2021-02-07.sch (EAGLE design)
At the start: 48 parts, among them J1 A-1JB, U0-C STM32F411CEUX, U0-S TPS62202, U1-S ICM-20948

Commit message: Finished Flight Ready PCB Draft
Parts:
- added JP2: (no value), pinhead:PINHD-1X5
- added LD1, LD2: (no value), adafruit:LEDCHIP-LED0805
- added R11, R12, R17: 10k, resistor:R-US_M0805
- added R13, R14, R15, R16: TBD, resistor:R-US_M0805
- added S2: (no value), switch-omron:10-XX
- added U$18, U$19: TLC5916SOIC-16, Computer2:TLC5916SOIC-16
- added U$20, U$21: TLC5926TSSOP, Computer2:TLC5926TSSOP
Connections:
- new net N$10: R15.1, U$20.R-EXT
- new net N$11: R16.1, U$21.R-EXT
- new net N$12: U$19.!OUT0!
- new net N$13: U$19.!OUT1!
- new net N$14: U$19.!OUT2!
- new net N$15: U$19.!OUT3
- new net N$16: U$19.!OUT7!
- new net N$17: U$19.!OUT6!
- new net N$18: U$19.!OUT5!
- new net N$19: U$19.!OUT4!
- new net N$20: U$18.!OUT0!
- new net N$21: U$18.!OUT1!
- new net N$22: U$18.!OUT2!
- new net N$23: U$18.!OUT3
- new net N$24: U$18.!OUT7!
- new net N$25: U$18.!OUT6!
- new net N$26: U$18.!OUT5!
- new net N$27: U$18.!OUT4!
- new net N$28: U$20.OUT15
- new net N$29: U$20.OUT14
- new net N$30: U$20.OUT13
- new net N$31: U$20.OUT12
- new net N$32: U$20.OUT11
- new net N$33: U$20.OUT10
- new net N$34: U$20.OUT9
- new net N$35: U$20.OUT8
- new net N$36: U$21.OUT15
- new net N$37: U$21.OUT14
- new net N$38: U$21.OUT13
- new net N$39: U$21.OUT12
- new net N$40: U$21.OUT11
- new net N$41: U$21.OUT10
- new net N$42: U$21.OUT9
- new net N$43: U$21.OUT8
- new net N$44: U$21.OUT0
- new net N$45: U$21.OUT1
- new net N$46: U$21.OUT2
- new net N$47: U$21.OUT3
- new net N$48: U$21.OUT4
- new net N$49: U$21.OUT5
- new net N$50: U$21.OUT6
- new net N$51: U$21.OUT7
- new net N$52: U$20.OUT0
- new net N$53: U$20.OUT1
- new net N$54: U$20.OUT2
- new net N$55: U$20.OUT3
- new net N$56: U$20.OUT4
- new net N$57: U$20.OUT5
- new net N$58: U$20.OUT6
- new net N$59: U$20.OUT7
- new net N$6: LD1.C, R11.1
- new net N$60: R17.1, S2.P1
- new net N$7: LD2.C, R12.1
- new net N$8: R13.1, U$18.R-EXT
- new net N$9: R14.1, U$19.R-EXT
- net 3V3: now also JP2.1, S2.S, U$18.VDD, U$19.VDD, U$20.VDD, U$21.VDD
- net BUTTON_IN: now also S2.P, U0-C.PA11; no longer U0-C.PA12
- net BUZZER_OUT: now also U0-C.PA12; no longer U0-C.PA11
- net GND: now also JP2.5, R11.2, R12.2, R13.2, R14.2, R15.2, R16.2, R17.2, U$18.!OE!(ED2), U$18.GND, U$19.!OE!(ED2), U$19.GND, U$20.!OE!(ED2), U$20.GND, U$21.!OE!(ED2), U$21.GND
- net LD1: now also LD1.A
- net LD2: now also LD2.A
- net SPI2B_LE: now also U$18.LE(ED1), U$19.LE(ED1), U$20.LE(ED1), U$21.LE(ED1)
- net SPI2B_MOSI: now also U$18.SDI, U$19.SDI, U$20.SDI, U$21.SDI
- net SPI2_CS0: now also U$4.2A; no longer U$4.4B
- net SPI2_CS2: now also U$4.4B; no longer U$4.2A
- net SPI2_SCK0: now also U$18.CLK, U$19.CLK, U$20.CLK, U$4.2Y; no longer U$4.4Y
- net SPI2_SCK2: now also U$4.4Y; no longer U$4.2Y
- net SPI2_SCK3: now also U$21.CLK
- net SWCLK: now also JP2.3
- net SWDIO: now also JP2.4
- net SWO: now also JP2.2
Other:
- note added: "IMU (SPI1 CS1)"
