File: PCBs/MITCH_2021-48/PSPS_AVNC_MITCH_2021-02-25.brd (EAGLE design)
At the start: 29.5 x 50.8 mm, 55 parts, among them J1 A-1JB, J2 1X2-3.5MM, U0-C STM32F411CEUX, U1-S ICM-20948, U11-S SN74LV1T34, U12-S SN74LV1T34, U13-S SN74LV1T34, U14-S SN74LV1T34, U14-S1 SN74LV1T34, U14-S2 SN74LV1T34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

Commit message: Continued refining MITCH 2021.0
Parts:
- added R10, R11, R9: (no value), resistor:R0805
- moved C1-0C 2.22 mm to (6.00, -3.62)
- moved C3-0C 2.22 mm to (8.12, -3.62)
- moved U11-S 0.75 mm to (5.25, -7.75)
- moved U12-S 0.75 mm to (1.75, -7.75)
- moved U13-S 0.75 mm to (-5.25, -7.75)
- moved U14-S 0.75 mm to (-1.75, -7.75)
- moved R3 0.62 mm to (10.2, -3.62)
- moved R4 0.62 mm to (10.2, -7.75)
- moved U$1 0.25 mm to (0.00, -3.25)
Connections:
- new net EXT_BATT: R11.2
- net BATT_MEAS: now also R10.2, R11.1
- net BUTTON_IN: now also R9.1
- net GND: now also R10.1, R9.2
Routing:
- net 3V3: track 141.9 -> 151.4 mm, vias 15 -> 16
- net BUTTON_IN: track 7.88 -> 15.4 mm, vias 1 -> 2
- net EXT_BATT: track 0.00 -> 2.70 mm, vias 0 -> 1
- net VCAP: track 7.93 -> 5.55 mm
- net BATT_MEAS: track 11.2 -> 9.62 mm
- net GND: track 250.0 -> 251.4 mm
- net N$15: track 19.8 -> 21.1 mm
- net VBAT: track 31.7 -> 33.0 mm
- net 1V8: track 28.4 -> 27.4 mm
- net SPI1_MISO: track 16.9 -> 17.8 mm
- net SPI1_MOSI: track 14.5 -> 13.6 mm, vias 2 -> 3
- net MOSI-1V8: track 6.69 -> 5.90 mm
- net CS_IMU: track 6.19 -> 6.02 mm, vias 1 -> 0
- net NRST: vias 4 -> 3
Other:
- board text added: "12mm coin cell can be added to help GPS acquire lock faster"
- board text added: "3V3"
- board text added: "ALA normal to PCB"
- board text added: "Apply insulation to shaded area"
- board text added: "B Elshimy"
- board text added: "B Wodetzki"
- board text added: "BATT MEAS"
- board text added: "BATT_MEAS"
- board text added: "BMP"
- board text added: "BUTTON"
- board text added: "BUZZER"
- board text added: "CS"
- board text added: "GPS"
- board text added: "GPS Ant."
- board text added: "IMU"
- board text added: "Improper use may destroy this device."
- board text added: "J Kaji"
- board text added: "J Wiley"
- board text added: "M Batistich"
- board text added: "M Paral"
- board text added: "MISO"
- board text added: "MOSI"
- board text added: "NRST"
- board text added: "R Horvath"
- board text added: "R1"
- board text added: "R2"
- board text added: "SCK"
- board text added: "SCL"
- board text added: "SDA"
- board text added: "SWCLK"
- board text added: "SWDIO"
- board text added: "SWO"
- board text added: "Storage"
- board text added: "Use provided voltage divider to protect the ADC."
- board text added: "V Vijay"
- board text added: "VDIV"
- board text added: "WARNING: BATT_MEAS cannot exceed 3.3V"

Commit message: Completed MITCH 2021.0 PCB. Ready for review
Parts:
- removed J2: 1X2-3.5MM, adafruit:1X2-3.5MM
Connections:
- net 3V3: no longer J2.2
- net GND: now also U1-S.20; no longer J2.1
Routing:
- net 3V3: track 151.4 -> 145.2 mm
- net GND: track 251.4 -> 248.3 mm
Other:
- board size 29.5 x 50.8 mm -> 25.4 x 50.8 mm
- board text removed: "+"
- board text removed: "+3.3V"
