File: PCBs/MITCH_2021-48/PSPS_AVNC_MITCH_2021-02-25.sch (EAGLE design)
At the start: 55 parts, among them J1 A-1JB, J2 1X2-3.5MM, U0-C STM32F411CEUX, U1-S ICM-20948, U11-S SN74LV1T34, U12-S SN74LV1T34, U13-S SN74LV1T34, U14-S SN74LV1T34, U14-S1 SN74LV1T34, U14-S2 SN74LV1T34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

Commit message: Continued refining MITCH 2021.0
Parts:
- added R10, R11, R9: (no value), resistor:R-US_R0805
Connections:
- new net EXT_BATT: R11.2
- net BATT_MEAS: now also R10.2, R11.1
- net BUTTON_IN: now also R9.1
- net GND: now also R10.1, R9.2
Changed lines of the file:
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@@
 <part name="GND21" library="supply1" library_urn="urn:adsk.eagle:library:371" deviceset="GND" device=""/>
 <part name="J2" library="adafruit" library_urn="urn:adsk.eagle:library:420" deviceset="1X2" device="-3.5MM" package3d_urn="urn:adsk.eagle:package:6240635/1"/>
+<part name="R9" library="resistor" library_urn="urn:adsk.eagle:library:348" deviceset="R-US_" device="R0805" package3d_urn="urn:adsk.eagle:package:23553/2"/>
+<part name="R10" library="resistor" library_urn="urn:adsk.eagle:library:348" deviceset="R-US_" device="R0805" package3d_urn="urn:adsk.eagle:package:23553/2"/>
+<part name="R11" library="resistor" library_urn="urn:adsk.eagle:library:348" deviceset="R-US_" device="R0805" package3d_urn="urn:adsk.eagle:package:23553/2"/>
+<part name="GND22" library="supply1" library_urn="urn:adsk.eagle:library:371" deviceset="GND" device=""/>
 </parts>
 <sheets>
@@
 <instance part="GND21" gate="1" x="27.94" y="-96.52" smashed="yes">
 <attribute name="VALUE" x="25.4" y="-99.06" size="1.778" layer="96"/>
+</instance>
+<instance part="R9" gate="G$1" x="68.58" y="-68.58" smashed="yes">
+<attribute name="NAME" x="64.77" y="-67.0814" size="1.778" layer="95"/>
+<attribute name="VALUE" x="64.77" y="-71.882" size="1.778" layer="96"/>
+</instance>
+<instance part="R10" gate="G$1" x="-30.48" y="-55.88" smashed="yes" rot="R90">
+<attribute name="NAME" x="-31.9786" y="-59.69" size="1.778" layer="95" rot="R90"/>
+<attribute name="VALUE" x="-27.178" y="-59.69" size="1.778" layer="96" rot="R90"/>
+</instance>
+<instance part="R11" gate="G$1" x="-30.48" y="-40.64" smashed="yes" rot="R90">
+<attribute name="NAME" x="-31.9786" y="-44.45" size="1.778" layer="95" rot="R90"/>
+<attribute name="VALUE" x="-27.178" y="-44.45" size="1.778" layer="96" rot="R90"/>
+</instance>
+<instance part="GND22" gate="1" x="-30.48" y="-63.5" smashed="yes">
+<attribute name="VALUE" x="-33.02" y="-66.04" size="1.778" layer="96"/>
 </instance>
 </instances>
@@
 <pinref part="GND21" gate="1" pin="GND"/>
 </segment>
+<segment>
+<pinref part="R9" gate="G$1" pin="2"/>
+<wire x1="73.66" y1="-68.58" x2="76.2" y2="-68.58" width="0.1524" layer="91"/>
+<label x="76.2" y="-68.58" size="1.27" layer="95" xref="yes"/>
+</segment>
+<segment>
+<pinref part="R10" gate="G$1" pin="1"/>
+<pinref part="GND22" gate="1" pin="GND"/>
+</segment>
 </net>
 <net name="SWDIO" class="0">
@@
 <label x="58.42" y="-17.78" size="1.27" layer="95" xref="yes"/>
 </segment>
+<segment>
+<pinref part="R9" gate="G$1" pin="1"/>
+<wire x1="63.5" y1="-68.58" x2="60.96" y2="-68.58" width="0.1524" layer="91"/>
+<label x="60.96" y="-68.58" size="1.27" layer="95" rot="R180" xref="yes"/>
+</segment>
 </net>
 <net name="BUZZER_OUT" class="0">
@@
 <wire x1="12.7" y1="-55.88" x2="12.7" y2="-58.42" width="0.1524" layer="91"/>
 <label x="12.7" y="-58.42" size="1.27" layer="95" rot="R270" xref="yes"/>
+</segment>
+<segment>
+<pinref part="R11" gate="G$1" pin="1"/>
+<pinref part="R10" gate="G$1" pin="2"/>
+<wire x1="-30.48" y1="-45.72" x2="-30.48" y2="-48.26" width="0.1524" layer="91"/>
+<wire x1="-30.48" y1="-48.26" x2="-30.48" y2="-50.8" width="0.1524" layer="91"/>
+<wire x1="-30.48" y1="-48.26" x2="-25.4" y2="-48.26" width="0.1524" layer="91"/>
+<junction x="-30.48" y="-48.26"/>
+<label x="-25.4" y="-48.26" size="1.27" layer="95" xref="yes"/>
 </segment>
 </net>
@@
 </segment>
 </net>
+<net name="EXT_BATT" class="0">
+<segment>
+<pinref part="R11" gate="G$1" pin="2"/>
+<wire x1="-30.48" y1="-35.56" x2="-30.48" y2="-33.02" width="0.1524" layer="91"/>
+<label x="-30.48" y="-33.02" size="1.27" layer="95" rot="R90" xref="yes"/>
+</segment>
+</net>

Commit message: Completed MITCH 2021.0 PCB. Ready for review
Parts:
- removed J2: 1X2-3.5MM, adafruit:1X2-3.5MM
Connections:
- net 3V3: no longer J2.2
- net GND: now also U1-S.RESV.GND; no longer J2.1
Changed lines of the file:
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@@
 <part name="C5-0C1" library="resistor" library_urn="urn:adsk.eagle:library:348" deviceset="C-US" device="C0805" package3d_urn="urn:adsk.eagle:package:23617/2" value="0.1uF"/>
 <part name="GND21" library="supply1" library_urn="urn:adsk.eagle:library:371" deviceset="GND" device=""/>
-<part name="J2" library="adafruit" library_urn="urn:adsk.eagle:library:420" deviceset="1X2" device="-3.5MM" package3d_urn="urn:adsk.eagle:package:6240635/1"/>
 <part name="R9" library="resistor" library_urn="urn:adsk.eagle:library:348" deviceset="R-US_" device="R0805" package3d_urn="urn:adsk.eagle:package:23553/2"/>
 <part name="R10" library="resistor" library_urn="urn:adsk.eagle:library:348" deviceset="R-US_" device="R0805" package3d_urn="urn:adsk.eagle:package:23553/2"/>
@@
 <attribute name="VALUE" x="180.34" y="27.94" size="1.778" layer="96"/>
 </instance>
-<instance part="J2" gate="G$1" x="91.44" y="50.8" smashed="yes"/>
 </instances>
 <busses>
@@
 </segment>
 <segment>
-<pinref part="J2" gate="G$1" pin="2"/>
 <wire x1="86.36" y1="50.8" x2="83.82" y2="50.8" width="0.1524" layer="91"/>
 <label x="83.82" y="50.8" size="1.27" layer="95" rot="R180" xref="yes"/>
@@
 </segment>
 <segment>
-<pinref part="J2" gate="G$1" pin="1"/>
 <wire x1="86.36" y1="53.34" x2="83.82" y2="53.34" width="0.1524" layer="91"/>
 <label x="83.82" y="53.34" size="1.27" layer="95" rot="R180" xref="yes"/>
 </segment>
-</net>
+<segment>
+<pinref part="U1-S" gate="G$1" pin="RESV.GND"/>
+<wire x1="-66.04" y1="147.32" x2="-66.04" y2="149.86" width="0.1524" layer="91"/>
+<label x="-66.04" y="149.86" size="1.27" layer="95" rot="R90" xref="yes"/>
+</segment>
+</net>
