File: MS5607 Breakout/MS5607 Breakout.sch (EAGLE design)
At the start: 58 parts, among them J1 A-1JB, J2 TFM-107-01-XXX-D-DS, U0-C STM32F411CEUX, U1-S ICM-20948, U11-S SN74LV1T34, U12-S SN74LV1T34, U13-S SN74LV1T34, U14-S SN74LV1T34, U14-S1 SN74LV1T34, U14-S2 SN74LV1T34, U2-S MMA1211KEG

Commit message: Improved Battery board interface nets
Parts:
- removed C1-0C, C1-0S1, C1-0S2: 4.7uF, resistor:C-USC0805
- removed C1-0S3: 22uF, resistor:C-USC0805
- removed C1-0S4, C1-1S, C2-0C, C2-1S, C3-0C, C3-1S, C4-0C, C5-0C, C5-0C1: 0.1uF, resistor:C-USC0805
- removed C1-0S5: 1uF, resistor:C-USC0805
- removed C1-0S6: 100uF, resistor:C-USC0805
- removed C1-0S7: 1nF, resistor:C-USC0805
- removed FB1-0C: MMZ2012Y152B, Computer2:MMZ2012Y152B
- removed J1: A-1JB, SamacSys_Parts:A-1JB
- removed J2: TFM-107-01-XXX-D-DS, TFM-107-01-XXX-D-DS:TFM-107-01-XXX-D-DS
- removed LED2, LED3, LED4, LED5: (no value), adafruit:LEDCHIPLED_0805
- removed R1-0C, R5, R6, R7, R8: 10k, resistor:R-US_R0805
- removed R1-C, R2-C, R3-C, R4-C, R4-C1: TBD, resistor:R-US_R0805
- removed R10, R11, R2, R3, R4, R9: (no value), resistor:R-US_R0805
- removed U$2: TC58CVG2S0HRAIJ, Computer2:TC58CVG2S0HRAIJ
- removed U$3: ASI09N27M-05Q, Computer2:ASI09N27M-05Q
- removed U$4: LTC1517ES5-5, Computer2:LTC1517ES5-5
- removed U$5: TLV74118PDBVR, Computer2:TLV74118PDBVR
- removed U$6: NPN_TRANSISTOR, Computer2:NPN_TRANSISTOR
- removed U$7: MS5607, Computer2:MS5607
- removed U$8: ULTIMATE_GPS, Computer2:ULTIMATE_GPS
- removed U0-C: STM32F411CEUX, Computer2:STM32F411CEUX
- removed U1-S: ICM-20948, Computer2:ICM-20948
- removed U11-S, U12-S, U13-S, U14-S, U14-S1, U14-S2: SN74LV1T34, Computer2:SN74LV1T34
- removed U2-S: MMA1211KEG, Computer2:MMA1211KEG
- added C1: (no value), resistor:C-USC0805
- added JP1: (no value), pinhead:PINHD-2X3
- U$1: value (none) -> MS5607; device adafruit:CR1220SMT -> Computer2:MS5607
Connections:
- removed net !RESET!: J2.5, U0-C.PB5
- removed net 1V8: C1-0S6.1, C3-1S.1, U$5.OUT, U1-S.VDDIO, U11-SG$1.VCC, U12-SG$1.VCC, U13-SG$1.VCC
- removed net 5V: C1-0S3.1, R8.2, U$3.V+, U$4.VOUT, U14-S2G$1.VCC, U2-S.VDD
- removed net ALA_MEAS: C1-0S7.1, R5.1, R6.2, U0-C.PA1
- removed net ALA_REF: R7.2, R8.1, U0-C.PA0
- removed net ALA_ST: U0-C.PB9, U14-S2G$2.A
- removed net ALA_STATUS: U0-C.PB8, U14-S1G$2.Y
- removed net BATT_MEAS: R10.2, R11.1, U0-C.PA4
- removed net BOOT0: R1-0C.2, U0-C.BOOT0
- removed net BUTTON_IN: J2.3, R9.1, U0-C.PA12
- removed net BUZZER_OUT: R1.1, U0-C.PA11
- removed net CS-1V8: U1-S.NCS, U11-SG$2.Y
- removed net CS_BMP: U$7.CSB@1, U$7.CSB@2, U0-C.PB10
- removed net CS_IMU: U0-C.PB2, U11-SG$2.A
- removed net CS_STORAGE: R2.1, U0-C.PA8
- removed net CS_STORAGE-VIA: J2.1, R2.2, U$2.!CS!
- removed net EXT_BATT: R11.2
- removed net I2C_SCL: J2.7, U0-C.PB6
- removed net I2C_SDA: J2.9, U0-C.PB7
- removed net LD1: R4-C.1, U0-C.PH0-OSC_IN
- removed net LD2: R3-C.1, U0-C.PC15
- removed net LD3: R2-C.1, U0-C.PC14
- removed net LD4: R1-C.1, U0-C.PC13
- removed net MISO-1V8: U1-S.SDO/AD0, U14-SG$2.A
- removed net MOSI-1V8: U1-S.SDA/SDI, U12-SG$2.Y
- removed net N$10: R3.1, U$1.+
- removed net N$11: R4-C1.2, U$3.V-, U$6.C
- removed net N$12: C1-0S4.1, U$4.C1+
- removed net N$13: C1-0S4.2, U$4.C1-
- removed net N$14: LED5.C, R4-C1.1
- removed net N$15: J1.SIGNAL, U$8.EX_ANT
- removed net N$16: R5.2, U2-S.VOUT
- removed net N$2: LED4.A, R4-C.2
- removed net N$3: LED3.A, R3-C.2
- removed net N$4: LED2.A, R2-C.2
- removed net N$5: LED1.A, R1-C.2
- removed net NRST: C5-0C1.1, J2.8, U0-C.NRST
- removed net SCK-1V8: U1-S.SCL/SCLK, U13-SG$2.Y
- removed net SPI1_MISO: U$7.SDO, U0-C.PA6, U14-SG$2.Y
- removed net SPI1_MOSI: U$7.SDI, U0-C.PA7, U12-SG$2.A
- removed net SPI1_SCK: U$7.SCLK, U0-C.PA5, U13-SG$2.A
- removed net SPI2_MISO: J2.4, U$2.SO/IO1, U0-C.PB14
- removed net SPI2_MOSI: J2.2, U$2.SI/IO0, U0-C.PB15
- removed net SPI2_SCK: J2.6, U$2.SCK, U0-C.PB13
- removed net ST-5V: U14-S2G$2.Y, U2-S.ST
- removed net STATUS-5V: U14-S1G$2.A, U2-S.STATUS
- removed net SWCLK: J2.12, U0-C.PA14
- removed net SWDIO: J2.10, U0-C.PA13
- removed net SWO: J2.14, U0-C.PB3
- removed net U1S-REGOUT: C1-1S.1, U1-S.REGOUT
- removed net USART2_RX: U$8.TX, U0-C.PA3
- removed net USART2_TX: U$8.RX, U0-C.PA2
- removed net VBAT: U$1.+1, U$8.VBACKUP, U0-C.VBAT
- removed net VBAT_MEAS: R3.2, R4.1, U0-C.PB0
- removed net VCAP: C1-0C.1, U0-C.VCAP_1
- removed net VREF+: C2-0C.1, FB1-0C.1, U0-C.VDDA/VREF+
- new net CS: JP1.6, U$1.CSB@1, U$1.CSB@2
- new net SCLK: JP1.3, U$1.SCLK
- new net SDI: JP1.4, U$1.SDI
- new net SDO: JP1.5, U$1.SDO
- net 3V3: now also C1.1, JP1.1, LED1.A, U$1.VDD; no longer C1-0S1.1, C1-0S2.1, C1-0S5.1, C2-1S.1, C3-0C.1, C4-0C.1, C5-0C.1, FB1-0C.2, J2.13, LED5.A, U$2.!HOLD!/IO3, U$2.!WP!/IO2, U$2.VCC, U$4.VIN, U$5.EN, U$5.IN, U$7.PS, U$7.VDD, U$8.VCC, U0-C.VDD@24, U0-C.VDD@36, U0-C.VDD@48, U1-S.VDD, U14-S1G$1.VCC, U14-SG$1.VCC
- net GND: now also C1.2, JP1.2, R1.2, U$1.GND, U$1.PS; no longer C1-0C.2, C1-0S1.2, C1-0S2.2, C1-0S3.2, C1-0S5.2, C1-0S6.2, C1-0S7.2, C1-1S.2, C2-0C.2, C2-1S.2, C3-0C.2, C3-1S.2, C4-0C.2, C5-0C.2, C5-0C1.2, J1.GND_1, J1.GND_2, J1.GND_3, J2.11, J2.15, J2.16, J2.17, J2.18, J2.19, J2.20, LED1.C, LED2.C, LED3.C, LED4.C, R1-0C.1, R10.1, R4.2, R6.1, R7.1, R9.2, U$1.-, U$2.VSS, U$4.GND, U$5.GND, U$6.E, U$7.GND, U$8.GND, U0-C.VSS, U0-C.VSS@23, U0-C.VSS@35, U0-C.VSS@47, U0-C.VSSA/VREF-, U1-S.GND, U1-S.RESV.GND, U11-SG$1.GND, U12-SG$1.GND, U13-SG$1.GND, U14-S1G$1.GND, U14-S2G$1.GND, U14-SG$1.GND, U2-S.VSS
- net N$1: now also LED1.C, R1.1; no longer R1.2, U$6.B
