File: PCBs/MITCH_2021-48/MITCH 2021-0 Production/PSPS_AVNC_MITCH_2021-0_PRODUCTION.sch (EAGLE design)
At the start: 58 parts, among them J1 A-1JB, J2 TFM-107-01-XXX-D-DS, U0-C STM32F411CEUX, U1-S ICM-20948, U11-S SN74LV1T34, U12-S SN74LV1T34, U13-S SN74LV1T34, U14-S SN74LV1T34, U14-S1 SN74LV1T34, U14-S2 SN74LV1T34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

Commit message: Improved Battery board interface nets
Parts:
- R2: value (none) -> 10k
Changed lines of the file:
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@@
 <part name="R1-0C" library="resistor" library_urn="urn:adsk.eagle:library:348" deviceset="R-US_" device="R0805" package3d_urn="urn:adsk.eagle:package:23553/2" value="10k"/>
 <part name="GND6" library="supply1" library_urn="urn:adsk.eagle:library:371" deviceset="GND" device=""/>
-<part name="R2" library="resistor" library_urn="urn:adsk.eagle:library:348" deviceset="R-US_" device="R0805" package3d_urn="urn:adsk.eagle:package:23553/2"/>
+<part name="R2" library="resistor" library_urn="urn:adsk.eagle:library:348" deviceset="R-US_" device="R0805" package3d_urn="urn:adsk.eagle:package:23553/2" value="10k"/>
 <part name="U1-S" library="Computer2" library_urn="urn:adsk.eagle:library:23762960" deviceset="ICM-20948" device="" package3d_urn="urn:adsk.eagle:package:12798673/2"/>
 <part name="U11-S" library="Computer2" library_urn="urn:adsk.eagle:library:23762960" deviceset="SN74LV1T34" device="" package3d_urn="urn:adsk.eagle:package:12825339/1"/>
