File: Battery Board/BatteryBoard.sch (EAGLE design)
At the start: 20 parts, among them IC1 MCP73831T-2ATI_OT, IC2 STM809TWX6F, J0 1725656, Q1 SQ2318BES-T1_GE3, U0 STM32L031K4U6

Commit message: Fixed the GND_OUT / 3V3 Nets
Parts:
- removed D1: GF1, diode:GF1
Connections:
- new net 3V3: C0.1, C1.1, C2.1, FB0.1, U0.VDD_1, U0.VDD_2
- net GND: no longer R0.2, U0.VSS
- net GND_OUT: now also R0.2, U0.VSS; no longer C0.1, C1.1, C2.1, FB0.1, U0.VDD_1, U0.VDD_2
- net NRST: no longer D1.A
- net PROTECTION_NRST: no longer D1.C
Other:
- note removed: "diode and mosfet parts need to be selected"
Changed lines of the file:
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@@
 <part name="C1" library="rcl" library_urn="urn:adsk.eagle:library:334" deviceset="C-US" device="C0805" package3d_urn="urn:adsk.eagle:package:23617/2" value="0.1uF"/>
 <part name="C0" library="rcl" library_urn="urn:adsk.eagle:library:334" deviceset="C-US" device="C0805" package3d_urn="urn:adsk.eagle:package:23617/2" value="0.1uF"/>
-<part name="GND1" library="supply1" library_urn="urn:adsk.eagle:library:371" deviceset="GND" device=""/>
 <part name="GND2" library="supply1" library_urn="urn:adsk.eagle:library:371" deviceset="GND" device=""/>
 <part name="C2" library="rcl" library_urn="urn:adsk.eagle:library:334" deviceset="C-US" device="C0805" package3d_urn="urn:adsk.eagle:package:23617/2" value="10uF"/>
@@
 <part name="C4" library="rcl" library_urn="urn:adsk.eagle:library:334" deviceset="C-US" device="C0805" package3d_urn="urn:adsk.eagle:package:23617/2" value="1uF"/>
 <part name="GND3" library="supply1" library_urn="urn:adsk.eagle:library:371" deviceset="GND" device=""/>
-<part name="GND4" library="supply1" library_urn="urn:adsk.eagle:library:371" deviceset="GND" device=""/>
 <part name="FB0" library="SamacSys_Parts" deviceset="MMZ2012Y152BTD25" device=""/>
 <part name="R1" library="rcl" library_urn="urn:adsk.eagle:library:334" deviceset="R-US_" device="R0805" package3d_urn="urn:adsk.eagle:package:23553/2"/>
@@
 <part name="GND12" library="supply1" library_urn="urn:adsk.eagle:library:371" deviceset="GND" device=""/>
 <part name="Q1" library="SamacSys_Parts" deviceset="SQ2318BES-T1_GE3" device=""/>
-<part name="D1" library="diode" library_urn="urn:adsk.eagle:library:210" deviceset="GF1" device="" package3d_urn="urn:adsk.eagle:package:43452/2"/>
+<part name="GND11" library="supply1" library_urn="urn:adsk.eagle:library:371" deviceset="GND" device=""/>
 </parts>
 <sheets>
 <sheet>
 <plain>
-<text x="86.36" y="35.56" size="1.27" layer="91">diode and mosfet parts need to be selected</text>
 </plain>
 <instances>
@@
 <attribute name="VALUE" x="-4.064" y="5.969" size="1.778" layer="96"/>
 </instance>
-<instance part="GND1" gate="1" x="33.02" y="86.36" smashed="yes" rot="R180">
-<attribute name="VALUE" x="35.56" y="88.9" size="1.778" layer="96" rot="R180"/>
-</instance>
 <instance part="GND2" gate="1" x="-5.08" y="0" smashed="yes">
 <attribute name="VALUE" x="-7.62" y="-2.54" size="1.778" layer="96"/>
@@
 <attribute name="VALUE" x="-25.4" y="-2.54" size="1.778" layer="96"/>
 </instance>
-<instance part="GND4" gate="1" x="27.94" y="73.66" smashed="yes" rot="R180">
-<attribute name="VALUE" x="30.48" y="76.2" size="1.778" layer="96" rot="R180"/>
-</instance>
 <instance part="FB0" gate="G$1" x="-38.1" y="0" smashed="yes" rot="R90">
 <attribute name="NAME" x="-45.72" y="16.51" size="1.778" layer="95" rot="R90" align="center-left"/>
@@
 <attribute name="VALUE" x="120.65" y="44.45" size="1.778" layer="96" align="center-left"/>
 </instance>
-<instance part="D1" gate="D" x="101.6" y="43.18" smashed="yes">
-<attribute name="NAME" x="99.06" y="45.72" size="1.778" layer="95"/>
-<attribute name="VALUE" x="99.06" y="39.37" size="1.778" layer="96"/>
+<instance part="GND11" gate="1" x="116.84" y="33.02" smashed="yes">
+<attribute name="VALUE" x="114.3" y="30.48" size="1.778" layer="96"/>
 </instance>
 </instances>
@@
 </net>
 <net name="GND" class="0">
-<segment>
-<pinref part="R0" gate="G$1" pin="2"/>
-<pinref part="GND1" gate="1" pin="GND"/>
-</segment>
 <segment>
 <pinref part="C0" gate="G$1" pin="2"/>
@@
 </segment>
 <segment>
-<pinref part="U0" gate="G$1" pin="VSS"/>
-<wire x1="27.94" y1="68.58" x2="27.94" y2="71.12" width="0.1524" layer="91"/>
-<pinref part="GND4" gate="1" pin="GND"/>
-</segment>
-<segment>
 <pinref part="R2" gate="G$1" pin="1"/>
 <pinref part="GND5" gate="1" pin="GND"/>
@@
 <segment>
 <pinref part="Q1" gate="G$1" pin="S"/>
-<wire x1="116.84" y1="38.1" x2="119.38" y2="38.1" width="0.1524" layer="91"/>
-<label x="119.38" y="38.1" size="1.27" layer="95" xref="yes"/>
-</segment>
-</net>
-<net name="GND_OUT" class="0">
-<segment>
-<pinref part="C0" gate="G$1" pin="1"/>
-<pinref part="C1" gate="G$1" pin="1"/>
-<wire x1="-5.08" y1="12.7" x2="2.54" y2="12.7" width="0.1524" layer="91"/>
-<wire x1="-5.08" y1="12.7" x2="-5.08" y2="15.24" width="0.1524" layer="91"/>
-<junction x="-5.08" y="12.7"/>
-<label x="-5.08" y="15.24" size="1.27" layer="95" rot="R90" xref="yes"/>
-<pinref part="C2" gate="G$1" pin="1"/>
-<wire x1="2.54" y1="12.7" x2="10.16" y2="12.7" width="0.1524" layer="91"/>
-<junction x="2.54" y="12.7"/>
-</segment>
-<segment>
-<pinref part="U0" gate="G$1" pin="VDD_1"/>
-<wire x1="15.24" y1="50.8" x2="12.7" y2="50.8" width="0.1524" layer="91"/>
-<label x="12.7" y="50.8" size="1.27" layer="95" rot="R180" xref="yes"/>
-</segment>
-<segment>
-<pinref part="U0" gate="G$1" pin="VDD_2"/>
-<wire x1="60.96" y1="33.02" x2="63.5" y2="33.02" width="0.1524" layer="91"/>
-<label x="63.5" y="33.02" size="1.27" layer="95" xref="yes"/>
-</segment>
-<segment>
-<pinref part="FB0" gate="G$1" pin="1"/>
-<wire x1="-38.1" y1="0" x2="-38.1" y2="-2.54" width="0.1524" layer="91"/>
-<label x="-38.1" y="-2.54" size="1.27" layer="95" rot="R270" xref="yes"/>
-</segment>
-<segment>
-<pinref part="Q1" gate="G$1" pin="D"/>
-<wire x1="116.84" y1="53.34" x2="116.84" y2="55.88" width="0.1524" layer="91"/>
-<label x="116.84" y="55.88" size="1.27" layer="95" xref="yes"/>
+<wire x1="116.84" y1="38.1" x2="116.84" y2="35.56" width="0.1524" layer="91"/>
+<pinref part="GND11" gate="1" pin="GND"/>
 </segment>
 </net>
@@
 <label x="12.7" y="43.18" size="1.27" layer="95" rot="R180" xref="yes"/>
 </segment>
-<segment>
-<pinref part="D1" gate="D" pin="A"/>
-<wire x1="99.06" y1="43.18" x2="96.52" y2="43.18" width="0.1524" layer="91"/>
-<label x="96.52" y="43.18" size="1.27" layer="95" rot="R180" xref="yes"/>
-</segment>
 </net>
 <net name="PROTECTION_NRST" class="0">
@@
 <wire x1="109.22" y1="43.18" x2="106.68" y2="43.18" width="0.1524" layer="91"/>
 <wire x1="106.68" y1="43.18" x2="106.68" y2="66.04" width="0.1524" layer="91"/>
-<pinref part="D1" gate="D" pin="C"/>
-<wire x1="106.68" y1="43.18" x2="104.14" y2="43.18" width="0.1524" layer="91"/>
-<junction x="106.68" y="43.18"/>
-</segment>
-</net>
+</segment>
+</net>
+<net name="GND_OUT" class="0">
+<segment>
+<pinref part="Q1" gate="G$1" pin="D"/>
+<wire x1="116.84" y1="53.34" x2="116.84" y2="55.88" width="0.1524" layer="91"/>
+<wire x1="116.84" y1="55.88" x2="119.38" y2="55.88" width="0.1524" layer="91"/>
+<label x="119.38" y="55.88" size="1.27" layer="95" xref="yes"/>
+</segment>
+<segment>
+<pinref part="U0" gate="G$1" pin="VSS"/>
+<wire x1="27.94" y1="68.58" x2="27.94" y2="71.12" width="0.1524" layer="91"/>
+<label x="27.94" y="71.12" size="1.27" layer="95" rot="R90" xref="yes"/>
+</segment>
+<segment>
+<pinref part="R0" gate="G$1" pin="2"/>
+<wire x1="33.02" y1="83.82" x2="33.02" y2="86.36" width="0.1524" layer="91"/>
+<label x="33.02" y="86.36" size="1.27" layer="95" rot="R90" xref="yes"/>
+</segment>
+</net>
+<net name="3V3" class="0">
+<segment>
+<pinref part="U0" gate="G$1" pin="VDD_1"/>
+<wire x1="15.24" y1="50.8" x2="12.7" y2="50.8" width="0.1524" layer="91"/>
+<label x="12.7" y="50.8" size="1.27" layer="95" rot="R180" xref="yes"/>
+</segment>
+<segment>
+<pinref part="C0" gate="G$1" pin="1"/>
+<pinref part="C1" gate="G$1" pin="1"/>
+<wire x1="-5.08" y1="12.7" x2="2.54" y2="12.7" width="0.1524" layer="91"/>
+<wire x1="-5.08" y1="12.7" x2="-5.08" y2="15.24" width="0.1524" layer="91"/>
+<junction x="-5.08" y="12.7"/>
+<label x="-5.08" y="15.24" size="1.27" layer="95" rot="R90" xref="yes"/>
+<pinref part="C2" gate="G$1" pin="1"/>
+<wire x1="2.54" y1="12.7" x2="10.16" y2="12.7" width="0.1524" layer="91"/>
+<junction x="2.54" y="12.7"/>
+</segment>
+<segment>
+<pinref part="FB0" gate="G$1" pin="1"/>
+<wire x1="-38.1" y1="0" x2="-38.1" y2="-2.54" width="0.1524" layer="91"/>
+<label x="-38.1" y="-2.54" size="1.27" layer="95" rot="R270" xref="yes"/>
+</segment>
+<segment>
+<pinref part="U0" gate="G$1" pin="VDD_2"/>
+<wire x1="60.96" y1="33.02" x2="63.5" y2="33.02" width="0.1524" layer="91"/>
+<label x="63.5" y="33.02" size="1.27" layer="95" xref="yes"/>
+</segment>
+</net>
