File: Battery Board/BatteryBoard.sch (EAGLE design)
At the start: 33 parts, among them IC1 TPS63060DSCT, J0 1725656, J1 1725669, J2 UJ2-MIBH2-4-SMT-TR, J3 MPTC-02-16-02-6.30-XX-X-V, J4 JSTPH2, J5 MPTC-02-04-02-6.30-XX-X-V-LC, Q1 IAUC60N04S6L030HATMA1, U0 STM32L031K4U6, U1 MCP73831T-2ATI_OT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

Commit message: Further PCB Routing
Connections:
- net GND: now also Q1.GND; no longer C0.2, C1.2, C2.2, C3.2, C4.2, J2.MH1, J2.MH2, J2.MH3, J2.MH4, R2.1
- net GND_OUT: now also C0.2, C1.2, C2.2, C3.2, C4.2, Q1.BATTERY_2, R2.1
Changed lines of the file:
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@@
 <part name="C1" library="rcl" library_urn="urn:adsk.eagle:library:334" deviceset="C-US" device="C0805" package3d_urn="urn:adsk.eagle:package:23617/2" value="0.1uF"/>
 <part name="C0" library="rcl" library_urn="urn:adsk.eagle:library:334" deviceset="C-US" device="C0805" package3d_urn="urn:adsk.eagle:package:23617/2" value="0.1uF"/>
-<part name="GND2" library="supply1" library_urn="urn:adsk.eagle:library:371" deviceset="GND" device=""/>
 <part name="C2" library="rcl" library_urn="urn:adsk.eagle:library:334" deviceset="C-US" device="C0805" package3d_urn="urn:adsk.eagle:package:23617/2" value="10uF"/>
 <part name="C3" library="rcl" library_urn="urn:adsk.eagle:library:334" deviceset="C-US" device="C0805" package3d_urn="urn:adsk.eagle:package:23617/2" value="0.1uF"/>
 <part name="C4" library="rcl" library_urn="urn:adsk.eagle:library:334" deviceset="C-US" device="C0805" package3d_urn="urn:adsk.eagle:package:23617/2" value="1uF"/>
-<part name="GND3" library="supply1" library_urn="urn:adsk.eagle:library:371" deviceset="GND" device=""/>
 <part name="FB0" library="SamacSys_Parts" deviceset="MMZ2012Y152BTD25" device=""/>
 <part name="R1" library="rcl" library_urn="urn:adsk.eagle:library:334" deviceset="R-US_" device="R0805" package3d_urn="urn:adsk.eagle:package:23553/2"/>
 <part name="R2" library="rcl" library_urn="urn:adsk.eagle:library:334" deviceset="R-US_" device="R0805" package3d_urn="urn:adsk.eagle:package:23553/2"/>
-<part name="GND5" library="supply1" library_urn="urn:adsk.eagle:library:371" deviceset="GND" device=""/>
 <part name="J0" library="SamacSys_Parts" deviceset="1725656" device=""/>
 <part name="GND6" library="supply1" library_urn="urn:adsk.eagle:library:371" deviceset="GND" device=""/>
@@
 <part name="J2" library="SamacSys_Parts" deviceset="UJ2-MIBH2-4-SMT-TR" device=""/>
 <part name="GND4" library="supply1" library_urn="urn:adsk.eagle:library:371" deviceset="GND" device=""/>
-<part name="GND13" library="supply1" library_urn="urn:adsk.eagle:library:371" deviceset="GND" device=""/>
 <part name="J3" library="MPTC-02-16-02-6.30-XX-X-V" deviceset="MPTC-02-16-02-6.30-XX-X-V" device=""/>
 <part name="GND14" library="supply1" library_urn="urn:adsk.eagle:library:371" deviceset="GND" device=""/>
@@
 <attribute name="VALUE" x="-4.064" y="5.969" size="1.778" layer="96"/>
 </instance>
-<instance part="GND2" gate="1" x="-5.08" y="0" smashed="yes">
-<attribute name="VALUE" x="-7.62" y="-2.54" size="1.778" layer="96"/>
-</instance>
 <instance part="C2" gate="G$1" x="10.16" y="10.16" smashed="yes">
 <attribute name="NAME" x="11.176" y="10.795" size="1.778" layer="95"/>
@@
 <attribute name="VALUE" x="-21.844" y="5.969" size="1.778" layer="96"/>
 </instance>
-<instance part="GND3" gate="1" x="-22.86" y="0" smashed="yes">
-<attribute name="VALUE" x="-25.4" y="-2.54" size="1.778" layer="96"/>
-</instance>
 <instance part="FB0" gate="G$1" x="-12.7" y="-12.7" smashed="yes">
 <attribute name="NAME" x="-6.35" y="-5.08" size="1.778" layer="95" align="center-left"/>
@@
 <attribute name="VALUE" x="-9.398" y="59.69" size="1.778" layer="96" rot="R90"/>
 </instance>
-<instance part="GND5" gate="1" x="-12.7" y="55.88" smashed="yes">
-<attribute name="VALUE" x="-15.24" y="53.34" size="1.778" layer="96"/>
-</instance>
 <instance part="J0" gate="G$1" x="-48.26" y="76.2" smashed="yes">
 <attribute name="NAME" x="-31.75" y="83.82" size="1.778" layer="95" align="center-left"/>
@@
 <instance part="GND4" gate="1" x="-25.4" y="86.36" smashed="yes">
 <attribute name="VALUE" x="-27.94" y="83.82" size="1.778" layer="96"/>
-</instance>
-<instance part="GND13" gate="1" x="-53.34" y="88.9" smashed="yes">
-<attribute name="VALUE" x="-55.88" y="86.36" size="1.778" layer="96"/>
 </instance>
 <instance part="J3" gate="G$1" x="-38.1" y="142.24" smashed="yes">
@@
 <net name="GND" class="0">
 <segment>
-<pinref part="C0" gate="G$1" pin="2"/>
-<pinref part="C1" gate="G$1" pin="2"/>
-<wire x1="-5.08" y1="5.08" x2="2.54" y2="5.08" width="0.1524" layer="91"/>
-<wire x1="-5.08" y1="5.08" x2="-5.08" y2="2.54" width="0.1524" layer="91"/>
-<junction x="-5.08" y="5.08"/>
-<pinref part="GND2" gate="1" pin="GND"/>
-<pinref part="C2" gate="G$1" pin="2"/>
-<wire x1="2.54" y1="5.08" x2="10.16" y2="5.08" width="0.1524" layer="91"/>
-<junction x="2.54" y="5.08"/>
-</segment>
-<segment>
-<pinref part="C4" gate="G$1" pin="2"/>
-<pinref part="C3" gate="G$1" pin="2"/>
-<wire x1="-22.86" y1="5.08" x2="-15.24" y2="5.08" width="0.1524" layer="91"/>
-<wire x1="-22.86" y1="5.08" x2="-22.86" y2="2.54" width="0.1524" layer="91"/>
-<junction x="-22.86" y="5.08"/>
-<pinref part="GND3" gate="1" pin="GND"/>
-</segment>
-<segment>
-<pinref part="R2" gate="G$1" pin="1"/>
-<pinref part="GND5" gate="1" pin="GND"/>
-</segment>
-<segment>
 <pinref part="J0" gate="G$1" pin="2"/>
 <pinref part="GND6" gate="1" pin="GND"/>
@@
 <pinref part="GND11" gate="1" pin="GND"/>
 <wire x1="162.56" y1="43.18" x2="162.56" y2="40.64" width="0.1524" layer="91"/>
+<pinref part="Q1" gate="A" pin="GND"/>
+<wire x1="160.02" y1="45.72" x2="160.02" y2="43.18" width="0.1524" layer="91"/>
+<junction x="160.02" y="43.18"/>
 </segment>
 <segment>
@@
 <wire x1="-25.4" y1="91.44" x2="-25.4" y2="88.9" width="0.1524" layer="91"/>
 <pinref part="GND4" gate="1" pin="GND"/>
-</segment>
-<segment>
-<pinref part="J2" gate="G$1" pin="MH1"/>
-<wire x1="-50.8" y1="101.6" x2="-53.34" y2="101.6" width="0.1524" layer="91"/>
-<wire x1="-53.34" y1="101.6" x2="-53.34" y2="99.06" width="0.1524" layer="91"/>
-<pinref part="J2" gate="G$1" pin="MH4"/>
-<wire x1="-53.34" y1="99.06" x2="-53.34" y2="96.52" width="0.1524" layer="91"/>
-<wire x1="-53.34" y1="93.98" x2="-53.34" y2="91.44" width="0.1524" layer="91"/>
-<wire x1="-50.8" y1="93.98" x2="-53.34" y2="93.98" width="0.1524" layer="91"/>
-<junction x="-53.34" y="93.98"/>
-<wire x1="-53.34" y1="93.98" x2="-53.34" y2="96.52" width="0.1524" layer="91"/>
-<pinref part="J2" gate="G$1" pin="MH2"/>
-<wire x1="-50.8" y1="99.06" x2="-53.34" y2="99.06" width="0.1524" layer="91"/>
-<junction x="-53.34" y="99.06"/>
-<pinref part="J2" gate="G$1" pin="MH3"/>
-<wire x1="-50.8" y1="96.52" x2="-53.34" y2="96.52" width="0.1524" layer="91"/>
-<junction x="-53.34" y="96.52"/>
-<pinref part="GND13" gate="1" pin="GND"/>
 </segment>
 <segment>
@@
 <wire x1="160.02" y1="50.8" x2="162.56" y2="50.8" width="0.1524" layer="91"/>
 <label x="162.56" y="50.8" size="1.27" layer="95" xref="yes"/>
-</segment>
-</net>
+<pinref part="Q1" gate="A" pin="BATTERY_2"/>
+<wire x1="160.02" y1="48.26" x2="160.02" y2="50.8" width="0.1524" layer="91"/>
+<junction x="160.02" y="50.8"/>
+</segment>
+<segment>
+<pinref part="C4" gate="G$1" pin="2"/>
+<pinref part="C3" gate="G$1" pin="2"/>
+<wire x1="-22.86" y1="5.08" x2="-15.24" y2="5.08" width="0.1524" layer="91"/>
+<wire x1="-22.86" y1="5.08" x2="-22.86" y2="2.54" width="0.1524" layer="91"/>
+<junction x="-22.86" y="5.08"/>
+<label x="-22.86" y="2.54" size="1.27" layer="95" rot="R270" xref="yes"/>
+</segment>
+<segment>
+<pinref part="C0" gate="G$1" pin="2"/>
+<pinref part="C1" gate="G$1" pin="2"/>
+<wire x1="-5.08" y1="5.08" x2="2.54" y2="5.08" width="0.1524" layer="91"/>
+<wire x1="-5.08" y1="5.08" x2="-5.08" y2="2.54" width="0.1524" layer="91"/>
+<junction x="-5.08" y="5.08"/>
+<pinref part="C2" gate="G$1" pin="2"/>
+<wire x1="2.54" y1="5.08" x2="10.16" y2="5.08" width="0.1524" layer="91"/>
+<junction x="2.54" y="5.08"/>
+<label x="-5.08" y="2.54" size="1.27" layer="95" rot="R270" xref="yes"/>
+</segment>
+<segment>
+<pinref part="R2" gate="G$1" pin="1"/>
+<wire x1="-12.7" y1="58.42" x2="-12.7" y2="55.88" width="0.1524" layer="91"/>
+<label x="-12.7" y="55.88" size="1.27" layer="95" rot="R270" xref="yes"/>
+</segment>
+</net>
