File: Battery Board/BatteryBoard.brd (EAGLE design)
At the start: 40.6 x 80.5 mm, 34 parts, among them IC1 TPS63060DSCT, J0 1725656, J1 1725669, J2 UJ2-MIBH2-4-SMT-TR, J3 MPTC-02-16-02-6.30-XX-X-V, J4 JSTPH2, J5 MPTC-02-04-02-6.30-XX-X-V-LC, Q1 IAUC60N04S6L030HATMA1, U0 STM32L031K4U6, U1 MCP73831T-2ATI_OT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

Commit message: minor additional routing
Routing:
- net SWDIO: track 10.3 -> 35.1 mm, vias 0 -> 2
- net SWCLK: track 12.5 -> 29.3 mm, vias 0 -> 2
- net I2C_SDA: track 78.3 -> 80.8 mm, vias 3 -> 4
- net I2C_SCL: track 85.6 -> 87.6 mm, vias 3 -> 4
- net NRST: vias 2 -> 3
- net GND: vias 14 -> 15
- net 3V3: vias 5 -> 6
Other:
- board text added: "RX"
- board text added: "TX"

Commit message: New transistor design started
Parts:
- added Q2: MMBTA56LT1G, transistor:SOT23-BEC
- added R10: 1M, rcl:R0805
- added R8, R9: 10k, rcl:R0805
- Q1: value IAUC60N04S6L030HATMA1 -> MMBTA56LT1G; device MarkParts:PG-TDSON-8-56 -> transistor:SOT23-BEC
- moved Q1 25.5 mm to (-19.6, -12.4), flipped to the top, turned to 0 degrees
Connections:
- removed net GND_OUT: C0.2, C1.2, C2.2, C3.2, C4.2, Q1.7, Q1.8, R0.2, R2.1, U0.33
- new net EN: IC1.3, Q1.E, Q2.E, R10.1
- new net N$2: Q1.B, R8.1
- new net N$4: Q2.B, R9.1
- net GND: now also C0.2, C1.2, C2.2, C3.2, C4.2, Q1.C, Q2.C, R0.2, R2.1, U0.33; no longer Q1.5, Q1.6
- net PROTECTION_NRST: now also R8.2; no longer Q1.1
- net SWITCH_IN: now also R9.2; no longer Q1.4
- net VBAT: now also R10.2; no longer IC1.3
Routing:
- net GND_OUT: track 35.3 -> 0.00 mm, vias 10 -> 0
- net GND: track 179.5 -> 213.3 mm, vias 15 -> 23
- net TX: track 54.2 -> 79.5 mm, vias 0 -> 3
- net RX: track 49.8 -> 74.7 mm, vias 0 -> 3
- net NRST: track 72.4 -> 92.9 mm, vias 3 -> 5
- net SWITCH_IN: track 6.14 -> 2.76 mm
- net PROTECTION_NRST: track 5.00 -> 1.86 mm
- net 3V3: track 90.8 -> 92.2 mm
- net VBAT: track 78.9 -> 78.2 mm
- net I2C_SCL: track 87.6 -> 88.3 mm
- removed copper zone on layer 1, net GND_OUT

Commit message: Battery Board work done
Parts:
- moved Q2 30.2 mm to (-2.79, 6.86), flipped to the bottom
- moved Q1 27.8 mm to (0.51, 6.86), flipped to the bottom
- moved R8 25.1 mm to (2.29, 3.05), flipped to the bottom, turned to 180 degrees
- moved R9 19.2 mm to (-1.02, 3.05), flipped to the bottom, turned to 270 degrees
- moved R10 18.9 mm to (-3.30, 3.05), flipped to the bottom, turned to 270 degrees
Routing:
- net GND: track 213.3 -> 229.7 mm, vias 23 -> 24
- net EN: track 0.00 -> 13.7 mm
- net P02: track 0.00 -> 10.7 mm
- net 3V3: track 92.2 -> 102.6 mm
- net SWITCH_IN: track 2.76 -> 8.82 mm, vias 0 -> 2
- net N$2: track 0.00 -> 2.76 mm
- net VBAT: track 78.2 -> 80.2 mm
- net N$4: track 0.00 -> 1.83 mm
- net PROTECTION_NRST: track 1.86 -> 2.95 mm
- net PA4: track 23.7 -> 22.9 mm

Commit message: further development. No airwires left
Routing:
- net NRST: track 92.9 -> 83.8 mm, vias 5 -> 8
- net 3V3: track 102.6 -> 106.6 mm
- net SWDIO: track 35.1 -> 32.6 mm, vias 2 -> 4
- net I2C_SCL: track 88.3 -> 85.9 mm
- net GND: track 229.7 -> 231.5 mm, vias 24 -> 21
- net I2C_SDA: track 81.1 -> 79.7 mm
- net RX: track 74.7 -> 76.0 mm
- net VBAT: track 80.2 -> 81.3 mm
- net TX: track 79.5 -> 80.4 mm, vias 3 -> 4
- net N$4: track 1.83 -> 2.56 mm
- net PA12: track 16.0 -> 15.3 mm, vias 2 -> 0
- net SWCLK: track 29.3 -> 28.8 mm, vias 2 -> 3
- added copper zone on layer 16, net I2C_SCL
- added copper zone on layer 16, net P02
- added copper zone on layer 1, net SWDIO

Commit message: Touch up before final review
Connections:
- net GND: now also IC1.11, IC1.12, IC1.13, IC1.14, IC1.15, IC1.16, IC1.17, IC1.18
Routing:
- net GND: track 231.5 -> 243.9 mm
- net 3V3: track 106.6 -> 105.4 mm

Commit message: Routed draft
Parts:
- moved R2 0.90 mm to (-7.49, 11.3)
- moved R1 0.77 mm to (-5.33, 11.3)
- moved C0 0.76 mm to (4.45, 12.1)
- moved C2 0.76 mm to (4.45, 9.78)
- moved C3 0.25 mm to (-3.17, 11.3)
- moved C1 0.25 mm to (-4.95, 18.9)
- moved R0 0.13 mm to (4.45, 15.1)
- moved C4 0.13 mm to (-1.02, 11.3)
- moved LED2 0.13 mm to (4.45, 17.0)
Connections:
- net I2C_SCL: now also J5.C01; no longer J5.D01
- net I2C_SDA: now also J5.D01; no longer J5.C01
Routing:
- net GND: track 243.9 -> 273.5 mm, vias 21 -> 15
- net NRST: track 83.8 -> 61.1 mm, vias 8 -> 4
- net VUSB: track 16.7 -> 35.7 mm
- net VBAT: track 81.3 -> 94.4 mm
- net I2C_SCL: track 85.9 -> 79.1 mm, vias 4 -> 3
- net I2C_SDA: track 79.7 -> 84.2 mm, vias 4 -> 3
- net 3V3: track 105.4 -> 101.8 mm, vias 6 -> 5
- net PB5: track 58.6 -> 61.2 mm
- net PA8: track 13.0 -> 14.8 mm, vias 2 -> 0
- net SWCLK: track 28.8 -> 30.5 mm, vias 3 -> 2
- net SWDIO: track 32.6 -> 34.0 mm, vias 4 -> 2
- net RX: track 76.0 -> 77.2 mm
- net TX: track 80.4 -> 81.5 mm
- net PA12: vias 0 -> 2
- added copper zone on layer 16, net VDDA
- removed copper zone on layer 16, net I2C_SCL
- removed copper zone on layer 1, net SWDIO

Commit message: Started shield
Routing:
- net GND: track 273.5 -> 272.5 mm
- added copper zone on layer 1, net 3V3
Changed lines of the file:
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@@
 <setting verticaltext="up"/>
 </settings>
-<grid distance="10" unitdist="mil" unit="mil" style="lines" multiple="1" display="yes" altdistance="5" altunitdist="mil" altunit="mil"/>
+<grid distance="10" unitdist="mil" unit="mil" style="lines" multiple="1" display="yes" altdistance="125" altunitdist="mil" altunit="mil"/>
 <layers>
 <layer number="1" name="Top" color="4" fill="1" visible="yes" active="yes"/>
@@
 </polygon>
 <wire x1="-11.505" y1="30.226" x2="-11.505" y2="29.539" width="1.016" layer="1"/>
-<wire x1="11.43" y1="30.226" x2="11.505" y2="30.226" width="1.016" layer="1"/>
 <via x="10.795" y="19.05" extent="1-16" drill="1"/>
 <contactref element="Q1" pad="C"/>
@@
 <wire x1="-11.505" y1="29.539" x2="-5.7714" y2="23.8054" width="1.016" layer="1"/>
 <via x="-0.955" y="17.973" extent="1-16" drill="0.35"/>
-<wire x1="-0.955" y1="17.973" x2="-0.762" y2="17.78" width="1.016" layer="16"/>
-<wire x1="-0.762" y1="17.78" x2="-0.762" y2="17.018" width="1.016" layer="16"/>
 <via x="5.395" y="9.779" extent="1-16" drill="0.35"/>
 <wire x1="5.395" y1="9.779" x2="5.6762" y2="10.0602" width="1.016" layer="1"/>
 <wire x1="5.6762" y1="10.0602" x2="5.6762" y2="11.938" width="1.016" layer="1"/>
-<wire x1="5.5492" y1="12.065" x2="5.6762" y2="11.938" width="1.016" layer="1"/>
-<wire x1="5.6762" y1="11.938" x2="5.522" y2="11.938" width="1.016" layer="1"/>
-<wire x1="5.522" y1="11.938" x2="5.395" y2="12.065" width="1.016" layer="1"/>
-<via x="5.395" y="12.065" extent="1-16" drill="0.35"/>
 <wire x1="5.6762" y1="11.938" x2="5.6762" y2="14.986" width="1.016" layer="1"/>
 <wire x1="5.495" y1="15.213" x2="5.495" y2="17.018" width="1.016" layer="16"/>
@@
 <wire x1="5.395" y1="15.113" x2="5.495" y2="15.213" width="0.6096" layer="16"/>
 <wire x1="5.6762" y1="16.29343125" x2="5.6762" y2="14.986" width="1.016" layer="1"/>
-<wire x1="-0.955" y1="17.973" x2="1.016" y2="17.973" width="1.016" layer="1"/>
-<wire x1="1.016" y1="17.973" x2="3.99663125" y2="17.973" width="1.016" layer="1"/>
+<wire x1="-0.955" y1="17.973" x2="3.99663125" y2="17.973" width="1.016" layer="1"/>
 <wire x1="3.99663125" y1="17.973" x2="5.6762" y2="16.29343125" width="1.016" layer="1"/>
+<wire x1="5.6762" y1="11.938" x2="5.5492" y2="12.065" width="0.2032" layer="1"/>
+<wire x1="5.5492" y1="12.065" x2="5.395" y2="12.065" width="0.2032" layer="1"/>
+<via x="5.395" y="12.065" extent="1-16" drill="0.35"/>
+<wire x1="-0.762" y1="17.78" x2="-0.955" y2="17.973" width="0.2032" layer="16"/>
 </signal>
 <signal name="VDDA">
@@
 <wire x1="-17.993" y1="29.423" x2="-15.6718" y2="27.1018" width="0.254" layer="16"/>
 <via x="8.255" y="13.97" extent="1-16" drill="1"/>
-<wire x1="-0.508" y1="15.326" x2="-0.512" y2="15.33" width="0.254" layer="16"/>
-<wire x1="-0.512" y1="15.33" x2="-0.512" y2="14.863" width="0.1778" layer="16"/>
 <via x="-0.254" y="14.3744" extent="1-16" drill="0.35"/>
 <wire x1="-0.512" y1="15.33" x2="-0.512" y2="14.6324" width="0.254" layer="16"/>
@@
 <contactref element="J3" pad="P03_4"/>
 <wire x1="5.08" y1="-8.128" x2="5.08" y2="-1.524" width="1.016" layer="1"/>
-<wire x1="-6.35" y1="30.071" x2="-6.505" y2="30.226" width="1.016" layer="16"/>
 <wire x1="0.992" y1="15.33" x2="0.988" y2="15.33" width="0.254" layer="16"/>
 <polygon width="0.254" layer="16" thermals="no">
@@
 <wire x1="6.8446" y1="9.56080625" x2="5.08" y2="7.79620625" width="1.016" layer="1"/>
 <wire x1="6.8446" y1="9.56080625" x2="6.8446" y2="15.24" width="1.016" layer="1"/>
-<wire x1="-4.953" y1="19.873" x2="-4.953" y2="19.8984" width="1.016" layer="16"/>
 <via x="-3.302" y="20.23" extent="1-16" drill="0.35"/>
 <wire x1="-3.302" y1="20.23" x2="-4.603" y2="21.531" width="1.016" layer="1"/>
@@
 <wire x1="3.495" y1="9.779" x2="5.08" y2="8.194" width="1.016" layer="1"/>
 <wire x1="5.08" y1="8.194" x2="5.08" y2="7.79620625" width="1.016" layer="1"/>
+<polygon width="0.2032" layer="1">
+<vertex x="3.937" y="-1.397"/>
+<vertex x="3.937" y="8.001"/>
+<vertex x="1.524" y="10.414"/>
+<vertex x="3.81" y="10.414"/>
+<vertex x="4.826" y="9.398"/>
+<vertex x="5.588" y="9.398"/>
+<vertex x="6.096" y="9.906"/>
+<vertex x="7.112" y="9.906"/>
+<vertex x="5.08" y="7.874"/>
+<vertex x="5.08" y="-8.382"/>
+<vertex x="3.048" y="-10.414"/>
+<vertex x="-3.556" y="-10.414"/>
+<vertex x="-3.81" y="-10.16"/>
+<vertex x="-3.81" y="-9.652"/>
+<vertex x="-3.048" y="-8.89"/>
+<vertex x="3.81" y="-8.89"/>
+<vertex x="4.7625" y="-7.9375"/>
+<vertex x="4.7625" y="-2.2225"/>
+</polygon>
+<polygon width="0.2032" layer="1">
+<vertex x="7.366" y="14.478"/>
+<vertex x="7.62" y="14.732"/>
+<vertex x="9.652" y="14.732"/>
+<vertex x="9.906" y="14.986"/>
+<vertex x="10.668" y="14.986"/>
+<vertex x="11.684" y="16.002"/>
+<vertex x="11.684" y="16.764"/>
+<vertex x="11.684" y="17.018"/>
+<vertex x="11.43" y="17.272"/>
+<vertex x="7.874" y="17.272"/>
+<vertex x="7.112" y="17.272"/>
+<vertex x="6.858" y="17.526"/>
+<vertex x="4.064" y="20.32"/>
+<vertex x="3.81" y="20.32"/>
+<vertex x="-1.016" y="20.32"/>
+<vertex x="-2.794" y="22.098"/>
+<vertex x="-4.064" y="23.368"/>
+<vertex x="-4.064" y="29.972"/>
+<vertex x="-5.08" y="30.988"/>
+<vertex x="-6.858" y="30.988"/>
+<vertex x="-7.366" y="30.48"/>
+<vertex x="-7.366" y="29.718"/>
+<vertex x="-7.366" y="26.416"/>
+<vertex x="-6.858" y="25.908"/>
+<vertex x="-5.08" y="24.13"/>
+<vertex x="-5.08" y="21.844"/>
+<vertex x="-5.08" y="21.59"/>
+<vertex x="-2.286" y="18.796"/>
+<vertex x="-2.032" y="18.542"/>
+<vertex x="4.318" y="18.542"/>
+<vertex x="6.35" y="16.51"/>
+<vertex x="6.35" y="10.16"/>
+<vertex x="5.588" y="9.398"/>
+<vertex x="6.096" y="8.89"/>
+<vertex x="6.858" y="9.652"/>
+<vertex x="6.858" y="11.43"/>
+<vertex x="6.858" y="13.97"/>
+</polygon>
 </signal>
 <signal name="N$12">
@@
 <wire x1="-0.6442" y1="23.62986875" x2="-0.6442" y2="23.114" width="0.2032" layer="16"/>
 <wire x1="-0.6442" y1="23.114" x2="-0.6442" y2="23.10613125" width="0.2032" layer="16"/>
-<wire x1="-0.062" y1="31.164" x2="-0.062" y2="24.21206875" width="0.2032" layer="16"/>
+<wire x1="-0.062" y1="31.164" x2="-0.062" y2="28.194" width="0.2032" layer="16"/>
+<wire x1="-0.062" y1="28.194" x2="-0.062" y2="24.21206875" width="0.2032" layer="16"/>
 <wire x1="-0.062" y1="24.21206875" x2="-0.6442" y2="23.62986875" width="0.2032" layer="16"/>
 <wire x1="1" y1="32.226" x2="-0.062" y2="31.164" width="0.2032" layer="16"/>
