File: MITCH_2021_SHIELD/ALA_BOARD.sch (EAGLE design)
At the start: 17 parts, among them J1 1725669, U1 NUCLEO-F401RE-BOTTOM, U2 TC58CVG2S0HRAIJ-ACTUAL, U3 MS5607_BREAKOUT, U4 SPARKFUN-9DOF-IMU, U5 SPARKFUN-BATTERY-BABYSITTER, U6 TPS63060DSCT

Commit message: further shield progress
Parts:
- removed C10: 10pF, rcl:C-USC0805
- removed C7: (2*10)uF, rcl:C-USC0805
- removed C8: (3*22)uF, rcl:C-USC0805
- removed C9: 0.1uF, rcl:C-USC0805
- removed J1: 1725669, SamacSys_Parts:1725669
- removed L1: XFL4020-102MEB, SamacSys_Parts:XFL4020-102MEB
- removed R5, R7: 1M, rcl:R-US_R0805
- removed R6: 111k, rcl:R-US_R0805
- removed S1: (no value), switch-omron:10-XX
- removed U2: TC58CVG2S0HRAIJ-ACTUAL, MITCH Shield:TC58CVG2S0HRAIJ-ACTUAL
- removed U3: MS5607_BREAKOUT, MITCH Shield:MS5607_BREAKOUT
- removed U4: SPARKFUN-9DOF-IMU, MITCH Shield:SPARKFUN-9DOF-IMU
- removed U5: SPARKFUN-BATTERY-BABYSITTER, MITCH Shield:SPARKFUN-BATTERY-BABYSITTER
- removed U6: TPS63060DSCT, SamacSys_Parts:TPS63060DSCT
- added C1: 1nF, rcl:C-USC0805
- added R1, R2, R3, R4: 10k 1%M, rcl:R-US_R0805
- U1: value NUCLEO-F401RE-BOTTOM -> MMA1211KEG; device MITCH Shield:NUCLEO-F401RE-BOTTOM -> MITCH Shield:MMA1211KEG
Connections:
- removed net 3V3: U1CN7.+3V3_S1, U2.!HOLD!/IO3, U2.!WP!/IO2, U2.VCC, U3.VIN, U4.VIN@2, U5.VPU
- removed net FB: C10.1, R5.1, R6.2, U6.FB
- removed net GPS_RX: U1CN10.PA10
- removed net GPS_TX: U1CN10.PA9
- removed net I2C_SCL: U1CN10.PB8, U5.SCL
- removed net I2C_SDA: U1CN10.PB9, U5.SDA
- removed net L1: L1.2, U6.L1
- removed net L2: L1.1, U6.L2
- removed net N$1: U1CN12.CNXX_1, U1CN12.CNXX_2
- removed net N$3: U1CN11.CNXX_1, U1CN11.CNXX_2
- removed net N$4: S1.S1, U5.CE
- removed net PG: R7.1, U6.PG
- removed net SENSORS_CS1: U1CN10.PC8, U3.CS
- removed net SENSORS_CS2: U1CN10.PC9, U4.NC
- removed net SENSORS_MISO: U1CN7.PC11, U3.SDO, U4.AD0
- removed net SENSORS_MOSI: U1CN7.PC12, U3.SDA, U4.DA
- removed net SENSORS_SCK: U1CN7.PC10, U3.SCL, U4.CL
- removed net STORAGE_CS: U1CN10.PB1, U2.!CS!
- removed net STORAGE_MISO: U1CN10.PB14, U2.SO/IO1
- removed net STORAGE_MOSI: U1CN10.PB15, U2.SI/IO0
- removed net STORAGE_SCK: U1CN10.PB13, U2.SCK
- removed net UART_RX: U1CN10.PA12
- removed net UART_TX: U1CN10.PA11
- removed net VAUX: C9.1, U6.VAUX
- removed net VBS: J1.1, U5.VOUT
- removed net VBS_SWITCH: C7.1, J1.2, U6.EN, U6.VIN
- new net VOUT: R3.1, U1.VOUT
- net 5V: now also R1.2, U1.VDD; no longer C8.1, R5.2, R7.2, U1CN7.E5V, U6.VOUT
- net ALA_MEAS: now also C1.1, R3.2, R4.2; no longer U1CN7.PC0/PB8
- net ALA_REF: now also R1.1, R2.2; no longer U1CN7.PC1/PB9
- net ALA_ST: now also U1.ST; no longer U1CN7.PC3
- net ALA_STATUS: now also U1.STATUS; no longer U1CN7.PC2
- net GND: now also C1.2, R2.1, R4.1, U1.VSS; no longer C10.2, C7.2, C8.2, C9.2, J1.3, R6.1, S1.P1, U1CN10.GND_S2, U1CN7.GND_S1, U2.VSS, U3.GND, U3.PS, U4.GND@1, U4.GND@2, U5.GND@1, U5.GND@2, U6.EP/PGND_1, U6.EP/PGND_2, U6.EP/PGND_3, U6.EP/PGND_4, U6.EP/PGND_5, U6.EP/PGND_6, U6.EP/PGND_7, U6.EP/PGND_8, U6.EP/PGND_9, U6.GND, U6.PS/SYNC
Other:
- moved on the sheet: X1-1, X1-2, X1-3, X1-4, X1-5, X1-6
