File: MITCH_2021_SHIELD/MITCH_2021-0_SHIELD.sch (EAGLE design)
At the start: 17 parts, among them J1 1725669, U1 NUCLEO-F401RE-BOTTOM, U2 TC58CVG2S0HRAIJ-ACTUAL, U3 MS5607_BREAKOUT, U4 SPARKFUN-9DOF-IMU, U5 SPARKFUN-BATTERY-BABYSITTER, U6 TPS63060DSCT

Commit message: Shield ready for production?
Connections:
- net GND: now also J1.1; no longer J1.3
- net VBS: now also J1.3; no longer J1.1
Other:
- moved on the sheet: J1
Changed lines of the file:
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@@
 <drawing>
 <settings>
-<setting alwaysvectorfont="no"/>
+<setting alwaysvectorfont="yes"/>
 <setting verticaltext="up"/>
 </settings>
@@
 <attribute name="VALUE" x="91.44" y="157.48" size="1.778" layer="96"/>
 </instance>
-<instance part="J1" gate="G$1" x="106.68" y="121.92" smashed="yes">
-<attribute name="NAME" x="123.19" y="129.54" size="1.778" layer="95" align="center-left"/>
-<attribute name="VALUE" x="123.19" y="127" size="1.778" layer="96" align="center-left"/>
+<instance part="J1" gate="G$1" x="106.68" y="116.84" smashed="yes" rot="MR180">
+<attribute name="NAME" x="123.19" y="109.22" size="1.778" layer="95" rot="MR180" align="center-left"/>
+<attribute name="VALUE" x="123.19" y="111.76" size="1.778" layer="96" rot="MR180" align="center-left"/>
 </instance>
 <instance part="GND7" gate="1" x="104.14" y="111.76" smashed="yes">
@@
 </segment>
 <segment>
-<pinref part="J1" gate="G$1" pin="3"/>
-<wire x1="106.68" y1="116.84" x2="104.14" y2="116.84" width="0.1524" layer="91"/>
 <wire x1="104.14" y1="116.84" x2="104.14" y2="114.3" width="0.1524" layer="91"/>
 <pinref part="GND7" gate="1" pin="GND"/>
+<pinref part="J1" gate="G$1" pin="1"/>
+<wire x1="106.68" y1="116.84" x2="104.14" y2="116.84" width="0.1524" layer="91"/>
 </segment>
 </net>
@@
 </segment>
 <segment>
-<pinref part="J1" gate="G$1" pin="1"/>
-<wire x1="104.14" y1="121.92" x2="106.68" y2="121.92" width="0.1524" layer="91"/>
-<label x="104.14" y="121.92" size="1.27" layer="95" rot="R180" xref="yes"/>
-</segment>
-</net>
+<label x="101.6" y="121.92" size="1.27" layer="95" rot="R180" xref="yes"/>
+<pinref part="J1" gate="G$1" pin="3"/>
+<wire x1="101.6" y1="121.92" x2="106.68" y2="121.92" width="0.1524" layer="91"/>
+</segment>
+</net>
