File: MITCH_2021_SHIELD/ALA_BOARD.brd (EAGLE design)
At the start: 25.4 x 25.4 mm, 7 parts, among them U1 MMA1211KEG

Commit message: refined design
Other:
- board size 25.4 x 25.4 mm -> 27.9 x 27.9 mm
Changed lines of the file:
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@@
 <board>
 <plain>
-<wire x1="0" y1="0" x2="25.4" y2="0" width="0" layer="20"/>
-<wire x1="25.4" y1="0" x2="25.4" y2="25.4" width="0" layer="20"/>
-<wire x1="25.4" y1="25.4" x2="0" y2="25.4" width="0" layer="20"/>
-<wire x1="0" y1="25.4" x2="0" y2="0" width="0" layer="20"/>
+<wire x1="-1.27" y1="-1.27" x2="26.67" y2="-1.27" width="0" layer="20"/>
+<wire x1="26.67" y1="-1.27" x2="26.67" y2="26.67" width="0" layer="20"/>
+<wire x1="26.67" y1="26.67" x2="-1.27" y2="26.67" width="0" layer="20"/>
+<wire x1="-1.27" y1="26.67" x2="-1.27" y2="-1.27" width="0" layer="20"/>
 <wire x1="10.16" y1="19.685" x2="10.16" y2="18.415" width="0.254" layer="21"/>
 <wire x1="14.224" y1="19.685" x2="14.224" y2="18.415" width="0.254" layer="21"/>
