File: MITCH_2021_SHIELD/MITCH_2021-0_SHIELD.brd (EAGLE design)
At the start: 71.1 x 101.6 mm, 18 parts, among them J1 22-27-2021-02, J2 22-27-2021-02, U1 NUCLEO-F401RE-BOTTOM, U3 MS5607_BREAKOUT, U4 SPARKFUN-9DOF-IMU, U5 SPARKFUN-BATTERY-BABYSITTER, U7 TPS63060DSCT

Commit message: further shield progress
Parts:
- removed J2: 22-27-2021-02, con-molex:6410-02
- J1: value 22-27-2021-02 -> 1725669; device con-molex:6410-02 -> SamacSys_Parts:1725669
- moved U4 25.4 mm to (-26.7, -27.9), flipped to the bottom
- moved U3 22.9 mm to (3.17, -51.4), flipped to the bottom, turned to 90 degrees
- moved J1 2.84 mm to (-30.5, 41.9), turned to 270 degrees
- flipped S1 to the bottom
- renumbered U$1 to U2, U7 to U6
Connections:
- net GND: now also J1.3; no longer J1.2, J2.2
- net VBS_SWITCH: now also J1.2; no longer J2.1
Routing:
- net 3V3: track 117.9 -> 142.8 mm
- net SENSORS_MISO: track 63.3 -> 47.3 mm
- net SENSORS_MOSI: track 85.9 -> 75.3 mm, vias 0 -> 4
- net SENSORS_CS2: track 15.5 -> 25.3 mm
- net N$4: track 31.8 -> 36.3 mm
- net GND: track 415.8 -> 412.9 mm
- net SENSORS_CS1: track 47.9 -> 45.2 mm, vias 0 -> 2
- net VBS_SWITCH: track 57.4 -> 60.1 mm
- net SENSORS_SCK: track 58.0 -> 56.5 mm
- net VBS: track 82.3 -> 81.6 mm
- added copper zone on layer 1, net VBS_SWITCH
- removed copper zone on layer 1, net VBS
Other:
- board text added: "BAROMETER"
- board text added: "BATTERY BABYSITTER"
- board text added: "IMU"

Commit message: Shield ready for production?
Parts:
- moved J1 5.08 mm to (-30.5, 36.8), flipped to the bottom, turned to 90 degrees
- flipped X1 to the bottom
Connections:
- net GND: now also J1.1; no longer J1.3
- net VBS: now also J1.3; no longer J1.1
Routing:
- net GND: track 412.9 -> 420.3 mm
- net VBS_SWITCH: vias 1 -> 2
Other:
- board text added: "5V"
- board text added: "ALA_MEAS"
- board text added: "ALA_REF"
- board text added: "ALA_ST"
- board text added: "ALA_STATUS"
- board text added: "CHARGE ENABLE"
- board text added: "GND"
- board text added: "VBS"
- board text added: "VBS_SWITCH"

Commit message: refined design
Parts:
- moved U4 1.27 mm to (-26.7, -29.2)
Routing:
- net SENSORS_MOSI: track 75.3 -> 77.3 mm
- net GND: track 420.3 -> 421.5 mm
- net SENSORS_SCK: track 56.5 -> 56.0 mm
- net SENSORS_CS2: track 25.3 -> 25.8 mm
- net SENSORS_MISO: track 47.3 -> 46.7 mm
- net 3V3: track 142.9 -> 143.4 mm
Changed lines of the file:
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@@
 <setting verticaltext="up"/>
 </settings>
-<grid distance="50" unitdist="mil" unit="mil" style="lines" multiple="1" display="yes" altdistance="25" altunitdist="mil" altunit="mil"/>
+<grid distance="50" unitdist="mil" unit="mil" style="lines" multiple="1" display="yes" altdistance="5" altunitdist="mil" altunit="mil"/>
 <layers>
-<layer number="1" name="Top" color="4" fill="1" visible="no" active="yes"/>
+<layer number="1" name="Top" color="4" fill="1" visible="yes" active="yes"/>
 <layer number="2" name="Route2" color="16" fill="1" visible="no" active="no"/>
 <layer number="3" name="Route3" color="17" fill="1" visible="no" active="no"/>
@@
 <layer number="19" name="Unrouted" color="6" fill="1" visible="yes" active="yes"/>
 <layer number="20" name="Dimension" color="24" fill="1" visible="yes" active="yes"/>
-<layer number="21" name="tPlace" color="7" fill="1" visible="no" active="yes"/>
+<layer number="21" name="tPlace" color="7" fill="1" visible="yes" active="yes"/>
 <layer number="22" name="bPlace" color="7" fill="1" visible="yes" active="yes"/>
-<layer number="23" name="tOrigins" color="15" fill="1" visible="no" active="yes"/>
+<layer number="23" name="tOrigins" color="15" fill="1" visible="yes" active="yes"/>
 <layer number="24" name="bOrigins" color="15" fill="1" visible="yes" active="yes"/>
-<layer number="25" name="tNames" color="7" fill="1" visible="no" active="yes"/>
+<layer number="25" name="tNames" color="7" fill="1" visible="yes" active="yes"/>
 <layer number="26" name="bNames" color="7" fill="1" visible="yes" active="yes"/>
 <layer number="27" name="tValues" color="7" fill="1" visible="no" active="yes"/>
@@
 <layer number="37" name="tTest" color="7" fill="1" visible="no" active="yes"/>
 <layer number="38" name="bTest" color="7" fill="1" visible="no" active="yes"/>
-<layer number="39" name="tKeepout" color="4" fill="11" visible="no" active="yes"/>
+<layer number="39" name="tKeepout" color="4" fill="11" visible="yes" active="yes"/>
 <layer number="40" name="bKeepout" color="1" fill="11" visible="yes" active="yes"/>
-<layer number="41" name="tRestrict" color="4" fill="10" visible="no" active="yes"/>
+<layer number="41" name="tRestrict" color="4" fill="10" visible="yes" active="yes"/>
 <layer number="42" name="bRestrict" color="1" fill="10" visible="yes" active="yes"/>
 <layer number="43" name="vRestrict" color="2" fill="10" visible="no" active="yes"/>
@@
 <layer number="49" name="Reference" color="7" fill="15" visible="no" active="yes"/>
 <layer number="50" name="dxf" color="7" fill="1" visible="no" active="no"/>
-<layer number="51" name="tDocu" color="7" fill="1" visible="no" active="yes"/>
+<layer number="51" name="tDocu" color="7" fill="1" visible="yes" active="yes"/>
 <layer number="52" name="bDocu" color="7" fill="1" visible="yes" active="yes"/>
 <layer number="53" name="tGND_GNDA" color="7" fill="9" visible="no" active="no"/>
@@
 </element>
 <element name="U3" library="MITCH Shield" package="MS5607_BREAKOUT" value="MS5607_BREAKOUT" x="3.175" y="-51.435" smashed="yes" rot="MR90"/>
-<element name="U4" library="MITCH Shield" package="SPARKFUN-9DOF-IMU1" value="SPARKFUN-9DOF-IMU" x="-26.67" y="-27.94" smashed="yes" rot="MR180"/>
+<element name="U4" library="MITCH Shield" package="SPARKFUN-9DOF-IMU1" value="SPARKFUN-9DOF-IMU" x="-26.67" y="-29.21" smashed="yes" rot="MR180"/>
 <element name="U5" library="MITCH Shield" package="SPARKFUN-BATTERY-BABYSITTER" value="SPARKFUN-BATTERY-BABYSITTER" x="0" y="1.27" smashed="yes" rot="MR270"/>
 <element name="U1" library="MITCH Shield" package="ST_NUCLEO-F401RE_BOTTOM" value="NUCLEO-F401RE-BOTTOM" x="0" y="-12.7" smashed="yes" rot="R180">
@@
 </polygon>
 <wire x1="11.2578" y1="-26.67" x2="11.4074" y2="-26.8196" width="1.016" layer="16"/>
-<wire x1="-17.78" y1="-29.21" x2="-15.24" y2="-26.67" width="1.016" layer="16"/>
-<wire x1="-15.24" y1="-26.67" x2="11.2578" y2="-26.67" width="1.016" layer="16"/>
+<wire x1="-17.78" y1="-30.48" x2="-13.97" y2="-26.67" width="1.016" layer="16"/>
+<wire x1="-13.97" y1="-26.67" x2="11.2578" y2="-26.67" width="1.016" layer="16"/>
 </signal>
 <signal name="GND">
@@
 <vertex x="34.29" y="44.45"/>
 </polygon>
-<wire x1="-20.32" y1="-52.07" x2="-20.32" y2="-44.45" width="1.016" layer="16"/>
-<wire x1="-20.32" y1="-44.45" x2="-20.32" y2="-29.21" width="1.016" layer="16"/>
+<wire x1="-20.32" y1="-53.34" x2="-20.32" y2="-44.45" width="1.016" layer="16"/>
+<wire x1="-20.32" y1="-44.45" x2="-20.32" y2="-30.48" width="1.016" layer="16"/>
 <wire x1="24.13" y1="-29.75776875" x2="24.13" y2="-30.2965875" width="0.254" layer="16"/>
 <wire x1="26.773" y1="-27.11476875" x2="24.13" y2="-29.75776875" width="0.254" layer="16"/>
@@
 <wire x1="19.1516" y1="29.3858125" x2="19.1516" y2="30.5816" width="1.016" layer="16"/>
 <wire x1="29.21" y1="40.64" x2="19.1516" y2="30.5816" width="1.016" layer="16"/>
-<wire x1="-20.32" y1="-29.21" x2="-20.32" y2="-26.35" width="1.016" layer="16"/>
+<wire x1="-20.32" y1="-30.48" x2="-20.32" y2="-26.35" width="1.016" layer="16"/>
 <wire x1="-20.32" y1="-26.35" x2="-16.51" y2="-22.54" width="1.016" layer="16"/>
 <wire x1="-20.32" y1="-44.45" x2="-3.81" y2="-44.45" width="1.016" layer="16"/>
@@
 <wire x1="5.207" y1="-40.64" x2="13.97" y2="-40.64" width="0.254" layer="1"/>
 <wire x1="13.97" y1="-40.64" x2="31.75" y2="-22.86" width="0.254" layer="1"/>
-<wire x1="-12.7" y1="-29.21" x2="-1.27" y2="-40.64" width="0.254" layer="1"/>
-<wire x1="-1.27" y1="-40.64" x2="5.207" y2="-40.64" width="0.254" layer="1"/>
+<wire x1="-12.7" y1="-30.48" x2="-2.54" y2="-40.64" width="0.254" layer="1"/>
+<wire x1="-2.54" y1="-40.64" x2="5.207" y2="-40.64" width="0.254" layer="1"/>
 </signal>
 <signal name="SENSORS_MOSI">
@@
 <wire x1="20.32" y1="-24.13" x2="19.05" y2="-25.4" width="0.254" layer="1"/>
 <via x="-8.89" y="-25.4" extent="1-16" drill="0.35"/>
-<wire x1="-8.89" y1="-25.4" x2="-12.7" y2="-25.4" width="0.254" layer="16"/>
-<via x="-12.7" y="-25.4" extent="1-16" drill="0.35"/>
-<wire x1="-12.7" y1="-25.4" x2="-15.24" y2="-27.94" width="0.254" layer="1"/>
-<wire x1="-15.24" y1="-27.94" x2="-15.24" y2="-29.21" width="0.254" layer="1"/>
+<wire x1="-8.89" y1="-25.4" x2="-13.97" y2="-25.4" width="0.254" layer="16"/>
+<via x="-13.97" y="-25.4" extent="1-16" drill="0.35"/>
+<wire x1="-13.97" y1="-25.4" x2="-15.24" y2="-26.67" width="0.254" layer="1"/>
+<wire x1="-15.24" y1="-26.67" x2="-15.24" y2="-30.48" width="0.254" layer="1"/>
 <wire x1="19.05" y1="-25.4" x2="-8.89" y2="-25.4" width="0.254" layer="1"/>
 </signal>
@@
 <wire x1="10.85223125" y1="-35.56" x2="23.55223125" y2="-22.86" width="0.254" layer="1"/>
 <wire x1="23.55223125" y1="-22.86" x2="29.21" y2="-22.86" width="0.254" layer="1"/>
-<wire x1="-10.16" y1="-29.21" x2="-3.81" y2="-35.56" width="0.254" layer="1"/>
-<wire x1="-3.81" y1="-35.56" x2="5.207" y2="-35.56" width="0.254" layer="1"/>
+<wire x1="-10.16" y1="-30.48" x2="-5.08" y2="-35.56" width="0.254" layer="1"/>
+<wire x1="-5.08" y1="-35.56" x2="5.207" y2="-35.56" width="0.254" layer="1"/>
 </signal>
 <signal name="SENSORS_CS1">
@@
 <wire x1="-31.75" y1="-22.86" x2="-27.94" y2="-26.67" width="0.254" layer="1"/>
 <wire x1="-27.94" y1="-26.67" x2="-27.94" y2="-31.75" width="0.254" layer="1"/>
-<wire x1="-27.94" y1="-31.75" x2="-25.4" y2="-34.29" width="0.254" layer="1"/>
-<wire x1="-25.4" y1="-34.29" x2="-10.16" y2="-34.29" width="0.254" layer="1"/>
-<via x="-10.16" y="-34.29" extent="1-16" drill="0.35"/>
-<wire x1="-10.16" y1="-34.29" x2="-3.81" y2="-34.29" width="0.254" layer="16"/>
-<via x="-3.81" y="-34.29" extent="1-16" drill="0.35"/>
-<wire x1="-3.81" y1="-34.29" x2="3.937" y2="-34.29" width="0.254" layer="1"/>
-<wire x1="3.937" y1="-34.29" x2="5.207" y2="-33.02" width="0.254" layer="1"/>
+<wire x1="-27.94" y1="-31.75" x2="-24.892" y2="-34.798" width="0.254" layer="1"/>
+<wire x1="-24.892" y1="-34.798" x2="-10.16" y2="-34.798" width="0.254" layer="1"/>
+<via x="-10.16" y="-34.798" extent="1-16" drill="0.35"/>
+<wire x1="-3.81" y1="-34.798" x2="-10.16" y2="-34.798" width="0.254" layer="16"/>
+<via x="-3.81" y="-34.798" extent="1-16" drill="0.35"/>
+<wire x1="-3.81" y1="-34.798" x2="3.429" y2="-34.798" width="0.254" layer="1"/>
+<wire x1="3.429" y1="-34.798" x2="5.207" y2="-33.02" width="0.254" layer="1"/>
 </signal>
 <signal name="SENSORS_CS2">
@@
 <wire x1="-29.21" y1="-22.86" x2="-27.94" y2="-21.59" width="0.254" layer="1"/>
 <wire x1="-27.94" y1="-21.59" x2="-22.86" y2="-21.59" width="0.254" layer="1"/>
-<wire x1="-20.32" y1="-24.13" x2="-12.7" y2="-24.13" width="0.254" layer="1"/>
-<wire x1="-12.7" y1="-24.13" x2="-7.62" y2="-29.21" width="0.254" layer="1"/>
+<wire x1="-20.32" y1="-24.13" x2="-13.97" y2="-24.13" width="0.254" layer="1"/>
+<wire x1="-13.97" y1="-24.13" x2="-7.62" y2="-30.48" width="0.254" layer="1"/>
 </signal>
 <signal name="I2C_SCL">
@@
 </signal>
 <signal name="N$2">
-<via x="-24.13" y="-30.48" extent="1-16" drill="2.9464"/>
+<via x="-24.13" y="-31.75" extent="1-16" drill="2.9464"/>
 </signal>
 <signal name="N$5">
-<via x="-24.13" y="-50.8" extent="1-16" drill="2.9464"/>
+<via x="-24.13" y="-52.07" extent="1-16" drill="2.9464"/>
 </signal>
 <signal name="N$6">
-<via x="-3.81" y="-50.8" extent="1-16" drill="2.9464"/>
+<via x="-3.81" y="-52.07" extent="1-16" drill="2.9464"/>
 </signal>
 <signal name="N$7">
-<via x="-3.81" y="-30.48" extent="1-16" drill="2.9464"/>
+<via x="-3.81" y="-31.75" extent="1-16" drill="2.9464"/>
 </signal>
 <signal name="N$8">
